File: 1_AP_Donat_Zeslovač/AP_zesilovac.sch (KiCad schematic (older format))
At the start: 50 parts, among them J1 AudioJack3, U1 TPA3116D2DADR-TPA3116D2DADR

Commit message: test
Parts:
- C13, C29: symbol Device:CP1 -> AP_zesilovac-rescue:CP1-Device
- U1: symbol tpa3116d2dadr-tpa3116d2dadr:TPA3116D2DADR-TPA3116D2DADR -> AP_zesilovac-rescue:TPA3116D2DADR-TPA3116D2DADR-tpa3116d2dadr-tpa3116d2dadr
Connections:
- net ZEM_JACKU is gone; now on net GND1: C5.2
- net GND: now also C10.2, C11.2, C14.1, Nulák1.1 (Pin_1); no longer C10.1, C11.1, C14.2, Nulák1.2 (Pin_2)
- net OUTNL: now also L4.1; no longer L4.2
- net VCC: now also C10.1, C11.1, C14.2, Nulák1.2 (Pin_2); no longer C10.2, C11.2, C14.1, Nulák1.1 (Pin_1)
- net at C18.2, C22.2, R8.2: now also L4.2; no longer L4.1
Other:
- moved on the sheet: C10, C11, C13, C14, C2, C23, C26, C29, L4, Nulák1, R2, RV1A
