File: 3_AP_Donat_Zeslovač/AP_zesilovac.sch (KiCad schematic (older format))
At the start: 50 parts, among them J1 AudioJack3, U1 TPA3116D2DADR-TPA3116D2DADR

Commit message: posledni_konrtrola
Changed lines of the file:
@@
 	1    0    0    -1
 $EndComp
-Connection ~ 1350 650
 $Comp
 L Device:R R5
@@
 Text GLabel 4450 1700 0    50   Input ~ 0
 13
-Text GLabel 1900 650  2    50   Input ~ 0
-15
-Text GLabel 4450 1800 0    50   Input ~ 0
-15
-Wire Wire Line
-	1350 650  1900 650
 Wire Notes Line
 	11150 550  11150 6450
@@
 Text GLabel 4450 3000 0    50   Input ~ 0
 4
-Text GLabel 4450 1600 0    50   Input ~ 0
-15
 Wire Wire Line
 	6050 3800 6050 3900
@@
 	5950 2100 6050 2100
 Wire Wire Line
-	4450 1600 4550 1600
-Wire Wire Line
 	4450 1700 4550 1700
-Wire Wire Line
-	4450 1800 4550 1800
 Wire Wire Line
 	4450 1900 4550 1900
@@
 Connection ~ 950  1850
 $Comp
-L power:GND2 #PWR?
+L power:GND2 #PWR0102
 U 1 1 60011567
 P 950 1950
-F 0 "#PWR?" H 950 1700 50  0001 C CNN
+F 0 "#PWR0102" H 950 1700 50  0001 C CNN
 F 1 "GND2" H 955 1777 50  0000 C CNN
 F 2 "" H 950 1950 50  0001 C CNN
@@
 	1    0    0    -1
 $EndComp
+Wire Wire Line
+	4100 1800 4100 1600
+Wire Wire Line
+	4100 1600 4550 1600
+Wire Wire Line
+	4100 1800 4550 1800
+Wire Wire Line
+	4100 1800 4100 1900
+Connection ~ 4100 1800
+$Comp
+L power:GND #PWR?
+U 1 1 600DED97
+P 4100 1900
+F 0 "#PWR?" H 4100 1650 50  0001 C CNN
+F 1 "GND" H 4105 1727 50  0000 C CNN
+F 2 "" H 4100 1900 50  0001 C CNN
+F 3 "" H 4100 1900 50  0001 C CNN
+	1    4100 1900
+	1    0    0    -1
+$EndComp
