File: 4_AP_Donat_Zeslovač/AP_zesilovac.kicad_pcb (KiCad board)
At the start: 2 copper layers, 50 parts, among them J1 AudioJack3, U1 TPA3116D2DADR-TPA3116D2DADR

Commit message: posledni_konrtrola
Routing:
- net GND: track 62.5 -> 64.4 mm, vias 5 -> 6
Other:
- board outline added: 65 x 52.8 mm
