File: 6_AP_Donat_Zeslovač/AP_zesilovac.kicad_pcb (KiCad board)
At the start: 2 copper layers, 50 parts, among them J1 AudioJack3, U1 TPA3116D2DADR-TPA3116D2DADR

Commit message: posledni_konrtrola
Parts:
- moved C14 54.3 mm to (143.3, 113.8), turned to 90 degrees
- moved C1 54.2 mm to (162.4, 105.3)
- moved C10 54.2 mm to (157.4, 111.8)
- moved C11 54.2 mm to (157.4, 114.3)
- moved C12 54.2 mm to (133.4, 104.3)
- moved C13 54.2 mm to (127.4, 110.3)
- moved C15 54.2 mm to (179.4, 79.3)
- moved C16 54.2 mm to (179.4, 90.3)
- moved C17 54.2 mm to (178.4, 101.3)
- moved C18 54.2 mm to (178.4, 114.5)
- moved C19 54.2 mm to (183.4, 79.3)
- moved C2 54.2 mm to (145.4, 79.3)
- moved C20 54.2 mm to (179.4, 95.3)
- moved C21 54.2 mm to (183.4, 101.3)
- moved C22 54.2 mm to (183.4, 114.3)
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Routing:
- net GND: track 72.0 -> 102.5 mm, vias 5 -> 12
- net (no net): vias 18 -> 16
Other:
- board outline added: 65 x 52.7 mm
